File: hardware/I2C_2_USB.sch (EAGLE design)
At the start: 13 parts, among them CN1 1X4-BIG, J3 USB-MICROB, U1 ATMEGA328P-MU-QFN32

Commit message: Add RST pushbutton, GND planes
Parts:
- added SW1: (no value), Seeed-OPL-Switch:SMD-BUTTON(2P-6.0X3.0X2.5MM)-DHT-1163S
Connections:
- net GND: now also SW1.2
- net RST: now also SW1.1
Changed lines of the file:
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@@
 <part name="+3V19" library="supply1" deviceset="+3V3" device=""/>
 <part name="P+2" library="supply1" deviceset="+5V" device=""/>
+<part name="SW1" library="Seeed-OPL-Switch" deviceset="SMD-BUTTON(2P-6.0X3.0X2.5MM)" device="-DHT-1163S"/>
+<part name="SUPPLY19" library="supply2" deviceset="GND" device=""/>
 </parts>
 <sheets>
@@
 <instance part="+3V19" gate="G$1" x="154.94" y="27.94"/>
 <instance part="P+2" gate="1" x="121.92" y="17.78" rot="R90"/>
+<instance part="SW1" gate="G$1" x="85.09" y="60.96" rot="R90"/>
+<instance part="SUPPLY19" gate="GND" x="85.09" y="74.93" rot="R180"/>
 </instances>
 <busses>
@@
 <pinref part="U$4" gate="G$1" pin="GND"/>
 <pinref part="SUPPLY27" gate="GND" pin="GND"/>
+</segment>
+<segment>
+<pinref part="SW1" gate="G$1" pin="2"/>
+<pinref part="SUPPLY19" gate="GND" pin="GND"/>
+<wire x1="85.09" y1="68.58" x2="85.09" y2="72.39" width="0.1524" layer="91"/>
 </segment>
 </net>
@@
 <segment>
 <pinref part="R7" gate="A" pin="1"/>
-<wire x1="86.36" y1="53.34" x2="82.55" y2="53.34" width="0.1524" layer="91"/>
+<wire x1="86.36" y1="53.34" x2="85.09" y2="53.34" width="0.1524" layer="91"/>
 <label x="82.55" y="53.34" size="1.27" layer="95" rot="R180" xref="yes"/>
+<pinref part="SW1" gate="G$1" pin="1"/>
+<wire x1="85.09" y1="53.34" x2="82.55" y2="53.34" width="0.1524" layer="91"/>
+<junction x="85.09" y="53.34"/>
 </segment>
 </net>

Commit message: Connect SDA and TxD Lines
Connections:
- net LED renamed LED_RED
- removed net ADCENA: U1.PB1(OC1A/PCINT1)
- removed net OUTA: U1.PB2(SS/OC1B/PCINT2)
- new net LED_BLUE: R2C.1, U1.PB2(SS/OC1B/PCINT2)
- new net LED_GREEN: R2B.1, U1.PB1(OC1A/PCINT1)
- net RXD: no longer R2C.1
- net TXD: no longer R2B.1
Changed lines of the file:
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@@
-</segment>
-</net>
-<net name="LED" class="0">
-<segment>
-<pinref part="U1" gate="G$1" pin="PB0(ICP/CLKO/PCINT0)"/>
-<wire x1="12.7" y1="99.06" x2="15.24" y2="99.06" width="0.1524" layer="91"/>
-<label x="15.24" y="99.06" size="1.27" layer="95" xref="yes"/>
-</segment>
-<segment>
-<wire x1="213.36" y1="68.58" x2="213.36" y2="63.5" width="0.1524" layer="91"/>
-<label x="213.36" y="63.5" size="1.27" layer="95" rot="R270" xref="yes"/>
-<pinref part="R2" gate="D" pin="1"/>
 </segment>
 </net>
@@
 </segment>
 </net>
-<net name="ADCENA" class="0">
-<segment>
-<pinref part="U1" gate="G$1" pin="PB1(OC1A/PCINT1)"/>
-<wire x1="12.7" y1="96.52" x2="15.24" y2="96.52" width="0.1524" layer="91"/>
-<label x="15.24" y="96.52" size="1.27" layer="95" xref="yes"/>
-</segment>
-</net>
 <net name="TXD" class="0">
 <segment>
@@
 <label x="15.24" y="48.26" size="1.27" layer="95" xref="yes"/>
 </segment>
-<segment>
-<wire x1="203.2" y1="68.58" x2="203.2" y2="63.5" width="0.1524" layer="91"/>
-<label x="203.2" y="63.5" size="1.27" layer="95" rot="R270" xref="yes"/>
-<pinref part="R2" gate="B" pin="1"/>
-</segment>
 </net>
 <net name="RXD" class="0">
@@
 <label x="15.24" y="50.8" size="1.27" layer="95" xref="yes"/>
 </segment>
-<segment>
-<wire x1="193.04" y1="68.58" x2="193.04" y2="63.5" width="0.1524" layer="91"/>
-<label x="193.04" y="63.5" size="1.27" layer="95" rot="R270" xref="yes"/>
-<pinref part="R2" gate="C" pin="1"/>
-</segment>
 </net>
 <net name="ADC" class="0">
@@
 <wire x1="12.7" y1="71.12" x2="15.24" y2="71.12" width="0.1524" layer="91"/>
 <label x="15.24" y="71.12" size="1.27" layer="95" xref="yes"/>
-</segment>
-</net>
-<net name="OUTA" class="0">
-<segment>
-<pinref part="U1" gate="G$1" pin="PB2(SS/OC1B/PCINT2)"/>
-<wire x1="12.7" y1="93.98" x2="15.24" y2="93.98" width="0.1524" layer="91"/>
-<label x="15.24" y="93.98" size="1.27" layer="95" xref="yes"/>
 </segment>
 </net>
@@
 </segment>
 </net>
+<net name="LED_GREEN" class="0">
+<segment>
+<pinref part="R2" gate="B" pin="1"/>
+<wire x1="203.2" y1="68.58" x2="203.2" y2="63.5" width="0.1524" layer="91"/>
+<label x="203.2" y="63.5" size="1.27" layer="95" rot="R270" xref="yes"/>
+</segment>
+<segment>
+<pinref part="U1" gate="G$1" pin="PB1(OC1A/PCINT1)"/>
+<wire x1="12.7" y1="96.52" x2="15.24" y2="96.52" width="0.1524" layer="91"/>
+<label x="15.24" y="96.52" size="1.27" layer="95" xref="yes"/>
+</segment>
+</net>
+<net name="LED_BLUE" class="0">
+<segment>
+<pinref part="R2" gate="C" pin="1"/>
+<wire x1="193.04" y1="68.58" x2="193.04" y2="63.5" width="0.1524" layer="91"/>
+<label x="193.04" y="63.5" size="1.27" layer="95" rot="R270" xref="yes"/>
+</segment>
+<segment>
+<pinref part="U1" gate="G$1" pin="PB2(SS/OC1B/PCINT2)"/>
+<wire x1="12.7" y1="93.98" x2="15.24" y2="93.98" width="0.1524" layer="91"/>
+<label x="15.24" y="93.98" size="1.27" layer="95" xref="yes"/>
+</segment>
+</net>
+<net name="LED_RED" class="0">
+<segment>
+<wire x1="213.36" y1="68.58" x2="213.36" y2="63.5" width="0.1524" layer="91"/>
+<label x="213.36" y="63.5" size="1.27" layer="95" rot="R270" xref="yes"/>
+<pinref part="R2" gate="D" pin="1"/>
+</segment>
+<segment>
+<pinref part="U1" gate="G$1" pin="PB0(ICP/CLKO/PCINT0)"/>
+<wire x1="12.7" y1="99.06" x2="15.24" y2="99.06" width="0.1524" layer="91"/>
+<label x="15.24" y="99.06" size="1.27" layer="95" xref="yes"/>
+</segment>
+</net>

Commit message: Add crypto module & backside labels
Parts:
- added U3: ATSHA204-TSU, SparkFun-IC-Special-Function:ATSHA204-TSU
Connections:
- new net CRYPTO: R7D.1, U3.SDA
- net +3V3: now also U3.VCC
- net GND: now also U3.GND
Other:
- note added: "pullup"
Changed lines of the file:
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@@
 <setting verticaltext="up"/>
 </settings>
-<grid distance="0.1" unitdist="inch" unit="inch" style="lines" multiple="1" display="no" altdistance="0.01" altunitdist="inch" altunit="inch"/>
+<grid distance="0.05" unitdist="inch" unit="inch" style="lines" multiple="1" display="no" altdistance="0.01" altunitdist="inch" altunit="inch"/>
 <layers>
 <layer number="1" name="Top" color="4" fill="1" visible="no" active="no"/>
@@
 <part name="SW1" library="Seeed-OPL-Switch" deviceset="SMD-BUTTON(2P-6.0X3.0X2.5MM)" device="-DHT-1163S"/>
 <part name="SUPPLY19" library="supply2" deviceset="GND" device=""/>
+<part name="U3" library="SparkFun-IC-Special-Function" deviceset="ATSHA204" device="-TSU"/>
+<part name="+3V10" library="supply1" deviceset="+3V3" device=""/>
+<part name="SUPPLY5" library="supply2" deviceset="GND" device=""/>
 </parts>
 <sheets>
@@
 <text x="205.74" y="63.5" size="1.27" layer="91" rot="R90">Green</text>
 <text x="215.138" y="63.5" size="1.27" layer="91">Red</text>
+<text x="137.16" y="-26.67" size="1.27" layer="91" rot="R90">pullup</text>
 </plain>
 <instances>
@@
 <instance part="SW1" gate="G$1" x="85.09" y="60.96" rot="R90"/>
 <instance part="SUPPLY19" gate="GND" x="85.09" y="74.93" rot="R180"/>
+<instance part="U3" gate="G$1" x="149.86" y="-31.75"/>
+<instance part="+3V10" gate="G$1" x="162.56" y="-26.67"/>
+<instance part="SUPPLY5" gate="GND" x="162.56" y="-36.83"/>
 </instances>
 <busses>
@@
 <pinref part="SUPPLY19" gate="GND" pin="GND"/>
 <wire x1="85.09" y1="68.58" x2="85.09" y2="72.39" width="0.1524" layer="91"/>
+</segment>
+<segment>
+<pinref part="U3" gate="G$1" pin="GND"/>
+<wire x1="157.48" y1="-34.29" x2="162.56" y2="-34.29" width="0.1524" layer="91"/>
+<pinref part="SUPPLY5" gate="GND" pin="GND"/>
 </segment>
 </net>
@@
 <wire x1="154.94" y1="25.4" x2="154.94" y2="17.78" width="0.1524" layer="91"/>
 </segment>
+<segment>
+<pinref part="U3" gate="G$1" pin="VCC"/>
+<wire x1="157.48" y1="-29.21" x2="162.56" y2="-29.21" width="0.1524" layer="91"/>
+<pinref part="+3V10" gate="G$1" pin="+3V3"/>
+</segment>
 </net>
 <net name="PUSH" class="0">
@@
 </segment>
 </net>
+<net name="CRYPTO" class="0">
+<segment>
+<pinref part="U3" gate="G$1" pin="SDA"/>
+<wire x1="139.7" y1="-31.75" x2="137.16" y2="-31.75" width="0.1524" layer="91"/>
+<label x="134.62" y="-31.75" size="1.27" layer="95" rot="R180" xref="yes"/>
+<wire x1="137.16" y1="-31.75" x2="134.62" y2="-31.75" width="0.1524" layer="91"/>
+<wire x1="137.16" y1="-29.21" x2="137.16" y2="-31.75" width="0.1524" layer="91"/>
+<junction x="137.16" y="-31.75"/>
+</segment>
+<segment>
+<pinref part="R7" gate="D" pin="1"/>
+<wire x1="86.36" y1="38.1" x2="82.55" y2="38.1" width="0.1524" layer="91"/>
+<label x="82.55" y="38.1" size="1.27" layer="95" rot="R180" xref="yes"/>
+</segment>
+</net>

Commit message: Add BLE module
Parts:
- added U2: RFD77101, SparkFun-RF:RFD77101
Connections:
- removed net RADIO_ON: U1.PD7(AIN1/PCINT23)
- new net BLE_RESET: U1.PD7(AIN1/PCINT23), U2.!RESET!
- net +3V3: now also U2.VDD
- net GND: now also U2.GND@44, U2.GND@45
- net RXD: now also U2.P0.00/AREF0
- net TXD: now also U2.P0.01/AIN2
Changed lines of the file:
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@@
 <part name="+3V10" library="supply1" deviceset="+3V3" device=""/>
 <part name="SUPPLY5" library="supply2" deviceset="GND" device=""/>
+<part name="U2" library="SparkFun-RF" deviceset="RFD77101" device=""/>
+<part name="SUPPLY1" library="supply2" deviceset="GND" device=""/>
+<part name="+3V1" library="supply1" deviceset="+3V3" device=""/>
 </parts>
 <sheets>
@@
 <instance part="+3V10" gate="G$1" x="162.56" y="-26.67"/>
 <instance part="SUPPLY5" gate="GND" x="162.56" y="-36.83"/>
+<instance part="U2" gate="G$1" x="226.06" y="-17.78"/>
+<instance part="SUPPLY1" gate="GND" x="241.3" y="-59.69"/>
+<instance part="+3V1" gate="G$1" x="187.96" y="1.27"/>
 </instances>
 <busses>
@@
 <wire x1="157.48" y1="-34.29" x2="162.56" y2="-34.29" width="0.1524" layer="91"/>
 <pinref part="SUPPLY5" gate="GND" pin="GND"/>
+</segment>
+<segment>
+<pinref part="U2" gate="G$1" pin="GND@44"/>
+<pinref part="SUPPLY1" gate="GND" pin="GND"/>
+<wire x1="241.3" y1="-50.8" x2="241.3" y2="-57.15" width="0.1524" layer="91"/>
+<pinref part="U2" gate="G$1" pin="GND@45"/>
+<wire x1="243.84" y1="-50.8" x2="241.3" y2="-50.8" width="0.1524" layer="91"/>
+<junction x="241.3" y="-50.8"/>
 </segment>
 </net>
@@
 <pinref part="+3V10" gate="G$1" pin="+3V3"/>
 </segment>
+<segment>
+<pinref part="U2" gate="G$1" pin="VDD"/>
+<pinref part="+3V1" gate="G$1" pin="+3V3"/>
+<wire x1="195.58" y1="-2.54" x2="187.96" y2="-2.54" width="0.1524" layer="91"/>
+<wire x1="187.96" y1="-2.54" x2="187.96" y2="-1.27" width="0.1524" layer="91"/>
+</segment>
 </net>
 <net name="PUSH" class="0">
@@
 <label x="15.24" y="48.26" size="1.27" layer="95" xref="yes"/>
 </segment>
+<segment>
+<pinref part="U2" gate="G$1" pin="P0.01/AIN2"/>
+<wire x1="223.52" y1="-50.8" x2="223.52" y2="-54.61" width="0.1524" layer="91"/>
+<label x="223.52" y="-54.61" size="1.27" layer="95" rot="R270" xref="yes"/>
+</segment>
 </net>
 <net name="RXD" class="0">
@@
 <label x="15.24" y="50.8" size="1.27" layer="95" xref="yes"/>
 </segment>
+<segment>
+<pinref part="U2" gate="G$1" pin="P0.00/AREF0"/>
+<wire x1="228.6" y1="-50.8" x2="228.6" y2="-54.61" width="0.1524" layer="91"/>
+<label x="228.6" y="-54.61" size="1.27" layer="95" rot="R270" xref="yes"/>
+</segment>
 </net>
 <net name="ADC" class="0">
@@
 <wire x1="12.7" y1="71.12" x2="15.24" y2="71.12" width="0.1524" layer="91"/>
 <label x="15.24" y="71.12" size="1.27" layer="95" xref="yes"/>
-</segment>
-</net>
-<net name="RADIO_ON" class="0">
-<segment>
-<pinref part="U1" gate="G$1" pin="PD7(AIN1/PCINT23)"/>
-<wire x1="12.7" y1="33.02" x2="15.24" y2="33.02" width="0.1524" layer="91"/>
-<label x="15.24" y="33.02" size="1.27" layer="95" xref="yes"/>
 </segment>
 </net>
@@
 </segment>
 </net>
+<net name="BLE_RESET" class="0">
+<segment>
+<pinref part="U2" gate="G$1" pin="!RESET!"/>
+<wire x1="195.58" y1="-5.08" x2="191.77" y2="-5.08" width="0.1524" layer="91"/>
+<label x="191.77" y="-5.08" size="1.27" layer="95" rot="R180" xref="yes"/>
+</segment>
+<segment>
+<pinref part="U1" gate="G$1" pin="PD7(AIN1/PCINT23)"/>
+<wire x1="12.7" y1="33.02" x2="15.24" y2="33.02" width="0.1524" layer="91"/>
+<label x="15.24" y="33.02" size="1.27" layer="95" xref="yes"/>
+</segment>
+</net>
